Commit message: update some files parameters and config files

File: install/bumperbot_description/share/bumperbot_description/urdf/bumperbot.urdf.xacro (robot description, xacro)
@@ -60,5 +60,5 @@
   </link>
   <joint name="wheel_right_joint" type="continuous">
-    <origin xyz="0 -0.0701101849418637 0" rpy="0 0 0" />
+    <origin xyz="0 -0.13 0" rpy="0 0 0" />
     <parent link="base_link" />
     <child link="wheel_right_link" />
@@ -89,5 +89,5 @@
   </link>
   <joint name="wheel_left_joint" type="continuous">
-    <origin xyz="0 0.0701101849418642 0" rpy="0 0 0" />
+    <origin xyz="0 0.13 0" rpy="0 0 0" />
     <parent link="base_link" />
     <child link="wheel_left_link" />
